Commit message: first commit

File: description/lidar.xacro (robot description, xacro)
@@ -4,5 +4,5 @@
         <parent link="chassis"/>
         <child link="laser_frame"/>
-        <origin xyz="0.122 0 0.212" rpy="0 0 0"/>
+        <origin xyz="0.050 0 0.135" rpy="0 0 0"/>
     </joint>
     <link name="laser_frame">
@@ -16,5 +16,5 @@
             <origin xyz="0 0 -0.05"/>
             <geometry>
-                <cylinder radius="0.01" length="0.1"/>
+                <cylinder radius="0.01" length="0.03"/>
             </geometry>
             <material name="black"/>

File: description/robot.urdf.xacro (robot description, xacro)
@@ -10,4 +10,4 @@
     </xacro:unless>
     <xacro:include filename="lidar.xacro" />
-    <xacro:include filename="camera.xacro" />
+    <!--xacro:include filename="camera.xacro" /-->
 </robot>

File: description/robot_core.xacro (robot description, xacro)
@@ -2,17 +2,17 @@
 <robot xmlns:xacro="http://www.ros.org/wiki/xacro" >
     <xacro:include filename="inertial_macros.xacro" />
-    <xacro:property name="chassis_length" value="0.335"/>
-    <xacro:property name="chassis_width" value="0.265"/>
-    <xacro:property name="chassis_height" value="0.138"/>
+    <xacro:property name="chassis_length" value="0.263"/>
+    <xacro:property name="chassis_width" value="0.193"/>
+    <xacro:property name="chassis_height" value="0.110"/>
     <xacro:property name="chassis_mass" value="1.0"/>
     <xacro:property name="wheel_radius" value="0.034"/>
     <xacro:property name="wheel_thickness" value="0.026"/>
     <xacro:property name="wheel_mass" value="0.05"/>
-    <xacro:property name="wheel_offset_x" value="0.226"/>
-    <xacro:property name="wheel_offset_y" value="0.166"/>
+    <xacro:property name="wheel_offset_x" value="0.168"/>
+    <xacro:property name="wheel_offset_y" value="0.111"/>
     <xacro:property name="wheel_offset_z" value="0.01"/>
     <xacro:property name="caster_wheel_radius" value="0.01"/>
     <xacro:property name="caster_wheel_mass" value="0.01"/>
-    <xacro:property name="caster_wheel_offset_x" value="0.075"/>
+    <xacro:property name="caster_wheel_offset_x" value="0.045"/>
     <xacro:property name="caster_wheel_offset_z" value="${wheel_offset_z - wheel_radius + caster_wheel_radius}"/>
     <material name="white">
